Commit message: Added lidar sensor

File: description/colors.xacro (robot description, xacro)
@@ -13,3 +13,6 @@
         <color rgba="0 0 0 1"/>
     </material>
+    <material name="red">
+        <color rgba="1 0 0 1"/>
+    </material>
 </robot>

File: description/gazebo_control.xacro (robot description, xacro)
@@ -1,5 +1,5 @@
 <?xml version="1.0"?>
 <robot xmlns:xacro="http://www.ros.org/wiki/xacro">
-    <xacro:include filename="robot_dims_params.xacro"/>
+    <xacro:include filename="robot_params.xacro"/>
     <gazebo>
         <plugin name="diff_drive" filename="libgazebo_ros_diff_drive.so">

File: description/robot.urdf.xacro (robot description, xacro)
@@ -5,3 +5,5 @@
     <!-- Include the gazebo control plugin that controls driving -->
     <xacro:include filename="gazebo_control.xacro" />
+    <!-- Include the lidar sensor -->
+    <xacro:include filename="lidar.xacro" />
 </robot>

File: description/robot_core.xacro (robot description, xacro)
@@ -4,5 +4,5 @@
     <xacro:include filename="inertial_macros.xacro"/>
     <xacro:include filename="colors.xacro"/>
-    <xacro:include filename="robot_dims_params.xacro"/>
+    <xacro:include filename="robot_params.xacro"/>
     <!-- BASE LINK -->
     <link name="base_link">

File: description/robot_params.xacro (robot description, xacro)
@@ -14,3 +14,12 @@
     <xacro:property name="wheel_mass" value="0.05"/>
     <xacro:property name="caster_wheel_mass" value="0.1"/>
+    <xacro:property name="laser_length" value="0.04"/>
+    <xacro:property name="laser_radius" value="0.05"/>
+    <xacro:property name="laser_mass" value="0.1"/>
+    <xacro:property name="laser_update_rate" value="10"/>
+    <xacro:property name="laser_samples" value="360"/>
+    <xacro:property name="laser_min_angle" value="-3.14"/>
+    <xacro:property name="laser_max_angle" value="3.14"/>
+    <xacro:property name="laser_min_range" value="0.3"/>
+    <xacro:property name="laser_max_range" value="12"/>
 </robot>
