Commit message: Added Basic Gazebo Sim + Modified Robot Dimensions

File: description/robot.urdf.xacro (robot description, xacro)
@@ -3,3 +3,5 @@
     <!-- Include the robot's core body description file -->
     <xacro:include filename="robot_core.xacro" />
+    <!-- Include the gazebo control plugin that controls driving -->
+    <xacro:include filename="gazebo_control.xacro" />
 </robot>

File: description/robot_core.xacro (robot description, xacro)
@@ -4,17 +4,5 @@
     <xacro:include filename="inertial_macros.xacro"/>
     <xacro:include filename="colors.xacro"/>
-    <!-- PARAMETERS -->
-    <xacro:property name="chassis_length" value="0.335"/>
-    <xacro:property name="chassis_width" value="0.265"/>
-    <xacro:property name="chassis_height" value="0.138"/>
-    <xacro:property name="wheel_offset_x" value="0.226"/>
-    <xacro:property name="wheel_radius" value="0.033"/>
-    <xacro:property name="wheel_thickness" value="0.026"/>
-    <xacro:property name="wheel_offset_y" value="0.1485"/>
-    <xacro:property name="caster_wheel_offset_x" value="0.075"/>
-    <xacro:property name="caster_wheel_radius" value="0.01"/>
-    <xacro:property name="chassis_mass" value="1.0"/>
-    <xacro:property name="wheel_mass" value="0.05"/>
-    <xacro:property name="caster_wheel_mass" value="0.01"/>
+    <xacro:include filename="robot_dims_params.xacro"/>
     <!-- BASE LINK -->
     <link name="base_link">
@@ -44,4 +32,7 @@
         </xacro:inertial_box>
     </link>
+    <gazebo reference="chassis">
+        <material>Gazebo/Orange</material>
+    </gazebo>
     <!-- LEFT WHEEL LINK -->
     <joint name="left_wheel_joint" type="continuous">
@@ -60,5 +51,5 @@
         <collision>
             <geometry>
-                <sphere radius="${wheel_radius}"/>
+                <cylinder radius="${wheel_radius}" length="${wheel_thickness}"/>
             </geometry>
         </collision>
@@ -67,4 +58,7 @@
         </xacro:inertial_cylinder>
     </link>
+    <gazebo reference="left_wheel">
+        <material>Gazebo/Blue</material>
+    </gazebo>
     <!-- RIGHT WHEEL LINK -->
     <joint name="right_wheel_joint" type="continuous">
@@ -83,5 +77,5 @@
         <collision>
             <geometry>
-                <sphere radius="${wheel_radius}"/>
+                <cylinder radius="${wheel_radius}" length="${wheel_thickness}"/>
             </geometry>
         </collision>
@@ -90,4 +84,7 @@
         </xacro:inertial_cylinder>
     </link>
+    <gazebo reference="right_wheel">
+        <material>Gazebo/Blue</material>
+    </gazebo>
     <!-- CASTER WHEEL LINK -->
     <joint name="caster_wheel_joint" type="fixed">
@@ -112,3 +109,8 @@
         </xacro:inertial_sphere>
     </link>
+    <gazebo reference="caster_wheel">
+        <material>Gazebo/White</material>
+        <mu1 value="0.001"/>
+        <mu2 value="0.001"/>
+    </gazebo>
 </robot>

Commit message: Added camera sensor

File: description/robot.urdf.xacro (robot description, xacro)
@@ -7,3 +7,5 @@
     <!-- Include the lidar sensor -->
     <xacro:include filename="lidar.xacro" />
+    <!-- Include the camera sensor -->
+    <xacro:include filename="camera.xacro" />
 </robot>

File: description/robot_params.xacro (robot description, xacro)
@@ -23,3 +23,12 @@
     <xacro:property name="laser_min_range" value="0.3"/>
     <xacro:property name="laser_max_range" value="12"/>
+    <xacro:property name="camera_length" value="0.01"/>
+    <xacro:property name="camera_width" value="0.03"/>
+    <xacro:property name="camera_height" value="0.03"/>
+    <xacro:property name="camera_update_rate" value="10"/>
+    <xacro:property name="camera_horizontal_fov" value="1.089"/>
+    <xacro:property name="camera_image_width" value="640"/>
+    <xacro:property name="camera_image_height" value="480"/>
+    <xacro:property name="camera_clip_near" value="0.05"/>
+    <xacro:property name="camera_clip_far" value="8.0"/>
 </robot>
