Commit message: added initial impl of gps navigation

File: src/alpr_bot/description/gazebo_control.xacro (robot description, xacro)
@@ -7,10 +7,11 @@
             <left_joint>left_wheel_joint</left_joint>
             <right_joint>right_wheel_joint</right_joint>
-            <wheel_separation>${wheel_offset_y * 2}</wheel_separation>
-            <wheel_diameter>${wheel_radius * 2}</wheel_diameter>
+            <wheel_separation>${wheel_separation}</wheel_separation>
+            <wheel_diameter>${wheel_diameter}</wheel_diameter>
             <!-- Limits -->
             <max_wheel_torque>200</max_wheel_torque>
             <max_wheel_acceleration>10.0</max_wheel_acceleration>
             <!-- Output -->
+            <odometry_topic>odom</odometry_topic>
             <odometry_frame>odom</odometry_frame>
             <robot_base_frame>base_link</robot_base_frame>
@@ -18,4 +19,11 @@
             <publish_odom_tf>true</publish_odom_tf>
             <publish_wheel_tf>true</publish_wheel_tf>
+            <ros>
+                <!--since gazebo_plugins publish tf topic in global namespace /tf only and it
+                cannot be remapped like (namespace/tf) through launch arguments -->
+                <remapping>/tf:=tf</remapping>
+            </ros>
+            <update_rate>30</update_rate>
+            <command_topic>cmd_vel</command_topic>
         </plugin>
     </gazebo>

File: src/alpr_bot/description/gps.xacro (robot description, xacro)
@@ -7,7 +7,5 @@
         <child link="gps_link"/>
         <origin xyz="${chassis_length/2} 0 ${chassis_length/2}" rpy="0 0 0"/>
-        <axis>
-          <xyz>0 0 1</xyz>
-        </axis>
+        <axis xyz="0 0 1"/>
     </joint>
     <link name="gps_link">
@@ -24,6 +22,6 @@
             </geometry>
         </collision>
-        <xacro:inertial_box mass="0.125" x="0.01" y="0.01" z="0.01">
-            <origin xyz="-0.052 0 0.111" rpy="0 0 0"/>
+        <xacro:inertial_box mass="${gps_mass}" x="0.01" y="0.01" z="0.01">
+            <origin xyz="${chassis_length/2} 0 ${chassis_length/2}" rpy="0 0 0"/>
         </xacro:inertial_box>
     </link>
@@ -31,6 +29,5 @@
         <sensor name="gps" type="gps">
           <always_on>true</always_on>
-          <update_rate>1</update_rate>
-          <pose>0 0 0 0 0 0</pose>
+          <update_rate>${gps_update_rate}</update_rate>
           <gps>
             <position_sensing>
@@ -38,5 +35,5 @@
                 <noise type="gaussian">
                   <mean>0.0</mean>
-                  <stddev>0.01</stddev>
+                  <stddev>${gps_noise_stddev}</stddev>
                 </noise>
               </horizontal>
@@ -44,5 +41,5 @@
                 <noise type="gaussian">
                   <mean>0.0</mean>
-                  <stddev>0.01</stddev>
+                  <stddev>${gps_noise_stddev}</stddev>
                 </noise>
               </vertical>

File: src/alpr_bot/description/imu.xacro (robot description, xacro)
@@ -6,14 +6,27 @@
         <child link="imu_link"/>
         <origin xyz="${chassis_length/2} 0 ${chassis_length/2}" rpy="0 0 0"/>
-        <axis>
-          <xyz>0 0 1</xyz>
-        </axis>
+        <axis xyz="0 0 1"/>
     </joint>
     <link name="imu_link">
+        <xacro:inertial_box mass="${imu_mass}" x="0.01" y="0.01" z="0.01">
+            <origin xyz="{chassis_length/2} 0 ${chassis_length/2}" rpy="0 0 0"/>
+        </xacro:inertial_box>
+        <visual>
+            <origin xyz="0 0 0" rpy="0 0 0"/>
+            <geometry>
+                <box size="0.01 0.01 0.01"/>
+            </geometry>
+        </visual>
+        <collision>
+            <origin xyz="0 0 0" rpy="0 0 0"/>
+            <geometry>
+                <box size="0.01 0.01 0.01"/>
+            </geometry>
+        </collision>
     </link>
     <gazebo reference="imu_link">
         <sensor name="imu" type="imu">
           <always_on>true</always_on>
-          <update_rate>200</update_rate>
+          <update_rate>${imu_update_rate}</update_rate>
           <imu>
             <angular_velocity>
@@ -21,5 +34,5 @@
                 <noise type="gaussian">
                   <mean>0.0</mean>
-                  <stddev>2e-4</stddev>
+                  <stddev>${imu_angular_velocity_stddev}</stddev>
                 </noise>
               </x>
@@ -27,5 +40,5 @@
                 <noise type="gaussian">
                   <mean>0.0</mean>
-                  <stddev>2e-4</stddev>
+                  <stddev>${imu_angular_velocity_stddev}</stddev>
                 </noise>
               </y>
@@ -33,5 +46,5 @@
                 <noise type="gaussian">
                   <mean>0.0</mean>
-                  <stddev>2e-4</stddev>
+                  <stddev>${imu_angular_velocity_stddev}</stddev>
                 </noise>
               </z>
@@ -41,5 +54,5 @@
                 <noise type="gaussian">
                   <mean>0.0</mean>
-                  <stddev>1.7e-2</stddev>
+                  <stddev>${imu_linear_acceleration_stddev}</stddev>
                 </noise>
               </x>
@@ -47,5 +60,5 @@
                 <noise type="gaussian">
                   <mean>0.0</mean>
-                  <stddev>1.7e-2</stddev>
+                  <stddev>${imu_linear_acceleration_stddev}</stddev>
                 </noise>
               </y>
@@ -53,5 +66,5 @@
                 <noise type="gaussian">
                   <mean>0.0</mean>
-                  <stddev>1.7e-2</stddev>
+                  <stddev>${imu_linear_acceleration_stddev}</stddev>
                 </noise>
               </z>

File: src/alpr_bot/description/lidar.xacro (robot description, xacro)
@@ -41,4 +41,9 @@
                     <max>${laser_max_range}</max>
                 </range>
+                <noise>
+                    <type>gaussian</type>
+                    <mean>${laser_noise_mean}</mean>
+                    <stddev>${laser_noise_stddev}</stddev>
+                </noise>
             </ray>
             <plugin name="laser_controller" filename="libgazebo_ros_ray_sensor.so">

File: src/alpr_bot/description/robot_core.xacro (robot description, xacro)
@@ -111,6 +111,6 @@
     <gazebo reference="caster_wheel">
         <material>Gazebo/White</material>
-        <mu1 value="0.001"/>
-        <mu2 value="0.001"/>
+        <mu1 value="0.01"/>
+        <mu2 value="0.01"/>
     </gazebo>
 </robot>

File: src/alpr_bot/description/robot_params.xacro (robot description, xacro)
@@ -2,29 +2,37 @@
 <robot xmlns:xacro="http://www.ros.org/wiki/xacro" >
     <!-- PARAMETERS -->
+    <!-- Robot Physical Dimensions -->
     <xacro:property name="chassis_length" value="0.3"/>
     <xacro:property name="chassis_width" value="0.3"/>
     <xacro:property name="chassis_height" value="0.15"/>
+    <xacro:property name="chassis_mass" value="0.5"/>
+    <xacro:property name="wheel_mass" value="0.05"/>
+    <xacro:property name="wheel_radius" value="0.05"/>
+    <xacro:property name="wheel_diameter" value="${wheel_radius * 2}"/>
+    <xacro:property name="wheel_thickness" value="0.04"/>
     <xacro:property name="wheel_offset_x" value="0.1"/>
-    <xacro:property name="wheel_radius" value="0.05"/>
-    <xacro:property name="wheel_thickness" value="0.04"/>
     <xacro:property name="wheel_offset_y" value="0.175"/>
+    <xacro:property name="wheel_separation" value="${wheel_offset_y * 2}"/>
     <xacro:property name="caster_wheel_offset_x" value="0.24"/>
     <xacro:property name="caster_wheel_radius" value="0.05"/>
-    <xacro:property name="chassis_mass" value="0.5"/>
-    <xacro:property name="wheel_mass" value="0.05"/>
     <xacro:property name="caster_wheel_mass" value="0.1"/>
+    <!-- LiDAR Parameters -->
+    <xacro:property name="laser_mass" value="0.1"/>
     <xacro:property name="laser_length" value="0.04"/>
     <xacro:property name="laser_radius" value="0.05"/>
-    <xacro:property name="laser_mass" value="0.1"/>
-    <xacro:property name="laser_update_rate" value="10"/>
+    <xacro:property name="laser_update_rate" value="5"/>
     <xacro:property name="laser_samples" value="360"/>
     <xacro:property name="laser_min_angle" value="-3.14"/>
     <xacro:property name="laser_max_angle" value="3.14"/>
-    <xacro:property name="laser_min_range" value="0.3"/>
+    <xacro:property name="laser_min_range" value="0.2"/>
     <xacro:property name="laser_max_range" value="12"/>
+    <xacro:property name="laser_noise_mean" value="0.0"/>
+    <xacro:property name="laser_noise_stddev" value="0.01"/>
+    <!-- Camera Parameters -->
+    <xacro:property name="camera_mass" value="0.03"/>
     <xacro:property name="camera_length" value="0.01"/>
     <xacro:property name="camera_width" value="0.03"/>
     <xacro:property name="camera_height" value="0.03"/>
-    <xacro:property name="camera_update_rate" value="10"/>
+    <xacro:property name="camera_update_rate" value="5"/>
     <xacro:property name="camera_horizontal_fov" value="1.089"/>
     <xacro:property name="camera_image_width" value="640"/>
@@ -32,3 +40,12 @@
     <xacro:property name="camera_clip_near" value="0.05"/>
     <xacro:property name="camera_clip_far" value="8.0"/>
+    <!-- GPS Parameters -->
+    <xacro:property name="gps_mass" value="0.05"/>
+    <xacro:property name="gps_update_rate" value="1"/>
+    <xacro:property name="gps_noise_stddev" value="0.01"/>
+    <!-- IMU Parameters -->
+    <xacro:property name="imu_mass" value="0.05"/>
+    <xacro:property name="imu_update_rate" value="200"/>
+    <xacro:property name="imu_angular_velocity_stddev" value="2e-4"/>
+    <xacro:property name="imu_linear_acceleration_stddev" value="1.7e-2"/>
 </robot>
