Commit message: added gps points follower

File: src/alpr_bot/description/camera.xacro (robot description, xacro)
@@ -30,5 +30,5 @@
         <sensor name="camera" type="camera">
             <pose> 0 0 0 0 0 0 </pose>
-            <visualize>true</visualize>
+            <visualize>false</visualize>
             <update_rate>${camera_update_rate}</update_rate>
             <camera>

File: src/alpr_bot/description/imu.xacro (robot description, xacro)
@@ -10,5 +10,5 @@
     <link name="imu_link">
         <xacro:inertial_box mass="${imu_mass}" x="0.01" y="0.01" z="0.01">
-            <origin xyz="{chassis_length/2} 0 ${chassis_length/2}" rpy="0 0 0"/>
+            <origin xyz="${chassis_length/2} 0 ${chassis_length/2}" rpy="0 0 0"/>
         </xacro:inertial_box>
         <visual>

File: src/alpr_bot/description/lidar.xacro (robot description, xacro)
@@ -27,5 +27,5 @@
         <sensor name="laser" type="ray">
             <pose> 0 0 0 0 0 0 </pose>
-            <visualize>true</visualize>
+            <visualize>false</visualize>
             <update_rate>${laser_update_rate}</update_rate>
             <ray>

File: src/alpr_bot/description/robot_core.xacro (robot description, xacro)
@@ -33,5 +33,5 @@
     </link>
     <gazebo reference="chassis">
-        <material>Gazebo/Orange</material>
+        <material>Gazebo/Test</material>
     </gazebo>
     <!-- LEFT WHEEL LINK -->

File: src/alpr_bot/description/robot_params.xacro (robot description, xacro)
@@ -3,12 +3,12 @@
     <!-- PARAMETERS -->
     <!-- Robot Physical Dimensions -->
-    <xacro:property name="chassis_length" value="0.3"/>
-    <xacro:property name="chassis_width" value="0.3"/>
-    <xacro:property name="chassis_height" value="0.15"/>
-    <xacro:property name="chassis_mass" value="0.5"/>
+    <xacro:property name="chassis_length" value="0.35"/>
+    <xacro:property name="chassis_width" value="0.35"/>
+    <xacro:property name="chassis_height" value="0.8"/>
+    <xacro:property name="chassis_mass" value="0.8"/>
     <xacro:property name="wheel_mass" value="0.05"/>
     <xacro:property name="wheel_radius" value="0.05"/>
     <xacro:property name="wheel_diameter" value="${wheel_radius * 2}"/>
-    <xacro:property name="wheel_thickness" value="0.04"/>
+    <xacro:property name="wheel_thickness" value="0.05"/>
     <xacro:property name="wheel_offset_x" value="0.1"/>
     <xacro:property name="wheel_offset_y" value="0.175"/>

Commit message: simulation demo

File: src/alpr_bot/description/camera.xacro (robot description, xacro)
@@ -5,5 +5,5 @@
         <parent link="chassis"/>
         <child link="camera_link"/>
-        <origin xyz="${chassis_length + camera_length/2} 0 ${3*chassis_height/4}" rpy="0 0 0"/>
+        <origin xyz="${chassis_length + camera_length/2} 0 ${chassis_height}" rpy="0 0 0"/>
     </joint>
     <link name="camera_link">

File: src/alpr_bot/description/robot_core.xacro (robot description, xacro)
@@ -33,5 +33,5 @@
     </link>
     <gazebo reference="chassis">
-        <material>Gazebo/Test</material>
+        <material>Gazebo/TIT</material>
     </gazebo>
     <!-- LEFT WHEEL LINK -->

File: src/alpr_bot/description/robot_params.xacro (robot description, xacro)
@@ -5,5 +5,5 @@
     <xacro:property name="chassis_length" value="0.35"/>
     <xacro:property name="chassis_width" value="0.35"/>
-    <xacro:property name="chassis_height" value="0.8"/>
+    <xacro:property name="chassis_height" value="0.55"/>
     <xacro:property name="chassis_mass" value="0.8"/>
     <xacro:property name="wheel_mass" value="0.05"/>
@@ -38,6 +38,6 @@
     <xacro:property name="camera_image_width" value="640"/>
     <xacro:property name="camera_image_height" value="480"/>
-    <xacro:property name="camera_clip_near" value="0.05"/>
-    <xacro:property name="camera_clip_far" value="8.0"/>
+    <xacro:property name="camera_clip_near" value="0.1"/>
+    <xacro:property name="camera_clip_far" value="20.0"/>
     <!-- GPS Parameters -->
     <xacro:property name="gps_mass" value="0.05"/>
